Commit message: add real robot control

File: fanuc_lrmate200id_support/urdf/lrmate200id7l_macro.xacro (robot description, xacro)
@@ -163,5 +163,5 @@
       </inertial>
     </link>
-	  <link name="${prefix}end_effector">
+	  <!-- <link name="${prefix}end_effector">
       <visual>
         <origin rpy="0 0 0" xyz="0 0 0"/>
@@ -176,5 +176,5 @@
       	<inertia ixx="1e-08" ixy="0" ixz="0" iyy="1e-08" iyz="0" izz="1e-08"/>
       </inertial>
-    </link>
+    </link> -->
 		<link name="world"/>
     <!-- joints: main serial chain -->
@@ -227,5 +227,5 @@
 			<dynamics damping="0.0" friction="1"/>
     </joint>
-		<joint name="${prefix}end_joint" type="revolute">
+		<!-- <joint name="${prefix}end_joint" type="revolute">
 			<origin xyz="0.021 0 0.0" rpy="0 1.5708 0"/>
       <parent link="${prefix}link_6"/>
@@ -234,5 +234,5 @@
       <limit effort="50" velocity="50" lower="0" upper="0" />
 			<dynamics damping="0.0" friction="1"/>
-    </joint>
+    </joint> -->
 		<joint name="${prefix}friction_plate_joint" type="fixed">
       <origin xyz="0.01 0 0" rpy="0 0 0" />
